File: hardware/skilleye_prototype/skilleye_regulator.kicad_sch (KiCad schematic)
At the start: 3 parts, among them U3 HT7833

Commit message: added MCU schematic + datasheets
Changed lines of the file:
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@@
 		(dnp no)
 		(property "Reference" "C5"
-			(at 153.4098 107.188 0)
+			(at 153.416 106.68 90)
 			(show_name no)
 			(do_not_autoplace no)
@@
 		)
 		(property "Value" "2.2uF"
-			(at 151.638 107.188 0)
+			(at 153.416 108.4518 90)
 			(show_name no)
 			(do_not_autoplace no)
@@
 		(dnp no)
 		(property "Reference" "C4"
-			(at 140.7098 107.188 0)
+			(at 136.398 106.68 90)
 			(show_name no)
 			(do_not_autoplace no)
@@
 		)
 		(property "Value" "1uF"
-			(at 138.938 107.188 0)
-			(show_name no)
-			(do_not_autoplace no)
+			(at 134.874 108.4518 90)
+			(show_name no)
+			(do_not_autoplace no)
