File: hardware/skilleye_1.0/skilleye_1.0.kicad_sch (KiCad schematic)
At the start: 3 parts, among them J2 USB_C_Receptacle_USB2.0_16P

Commit message: added 2.0 schematic
Parts:
- R11, R12: footprint (none) -> Resistor_SMD:R_0805_2012Metric
Changed lines of the file:
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@@
 			)
 		)
-		(property "Footprint" ""
+		(property "Footprint" "Resistor_SMD:R_0805_2012Metric"
 			(at 206.248 95.25 90)
 			(hide yes)
@@
 		)
 		(instances
-			(project "skilleye"
+			(project "skilleye_1.0"
 				(path "/e922ced9-cce7-4ffa-8992-2bb79546169b"
 					(reference "R11")
@@
 		)
 		(instances
-			(project "skilleye"
+			(project "skilleye_1.0"
 				(path "/e922ced9-cce7-4ffa-8992-2bb79546169b"
 					(reference "#PWR021")
@@
 		)
 		(instances
-			(project "skilleye"
+			(project "skilleye_1.0"
 				(path "/e922ced9-cce7-4ffa-8992-2bb79546169b"
 					(reference "#PWR023")
@@
 		)
 		(instances
-			(project "skilleye"
+			(project "skilleye_1.0"
 				(path "/e922ced9-cce7-4ffa-8992-2bb79546169b"
 					(reference "#PWR022")
@@
 		)
 		(instances
-			(project "skilleye"
+			(project "skilleye_1.0"
 				(path "/e922ced9-cce7-4ffa-8992-2bb79546169b"
 					(reference "J2")
@@
 		)
 		(instances
-			(project "skilleye"
+			(project "skilleye_1.0"
 				(path "/e922ced9-cce7-4ffa-8992-2bb79546169b"
 					(reference "#PWR024")
@@
 			)
 		)
-		(property "Footprint" ""
+		(property "Footprint" "Resistor_SMD:R_0805_2012Metric"
 			(at 207.772 95.25 90)
 			(hide yes)
@@
 		)
 		(instances
-			(project "skilleye"
+			(project "skilleye_1.0"
 				(path "/e922ced9-cce7-4ffa-8992-2bb79546169b"
 					(reference "R12")
@@
 		)
 		(instances
-			(project "skilleye"
+			(project "skilleye_1.0"
 				(path "/e922ced9-cce7-4ffa-8992-2bb79546169b"
 					(page "3")
@@
 		)
 		(instances
-			(project "skilleye"
+			(project "skilleye_1.0"
 				(path "/e922ced9-cce7-4ffa-8992-2bb79546169b"
 					(page "2")
@@
 		)
 		(instances
-			(project "skilleye"
+			(project "skilleye_1.0"
 				(path "/e922ced9-cce7-4ffa-8992-2bb79546169b"
 					(page "4")
