File: hardware/skilleye_1.0/skilleye_charging.kicad_sch (KiCad schematic)
At the start: 15 parts, among them J1 Conn_01x02_Pin, Q1 FS8205A, U1 TP4056-42-ESOP8, U2 DW01A

Commit message: added 2.0 schematic
Parts:
- C1, C2, C3: footprint (none) -> Capacitor_SMD:C_0805_2012Metric
- D1, D2: footprint (none) -> LED_SMD:LED_0805_2012Metric
- J1: footprint (none) -> Connector_PinHeader_2.54mm:PinHeader_1x02_P2.54mm_Vertical
- Q1: footprint (none) -> FS8205A:SOP65P640X120-8N
- R1, R2, R3, R4, R5, R6: footprint (none) -> Resistor_SMD:R_0805_2012Metric
- U1: footprint Package_SO:SOIC-8-1EP_3.9x4.9mm_P1.27mm_EP2.41x3.3mm_ThermalVias -> Package_SO:SOIC-8-1EP_3.9x4.9mm_P1.27mm_EP2.41x3.81mm
Changed lines of the file:
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@@
 		)
 		(instances
-			(project "skilleye"
+			(project "skilleye_1.0"
 				(path "/e922ced9-cce7-4ffa-8992-2bb79546169b/772fd356-96ac-42b2-8558-9fa39f1e8a4f"
 					(reference "#PWR01")
@@
 			)
 		)
-		(property "Footprint" ""
+		(property "Footprint" "Resistor_SMD:R_0805_2012Metric"
 			(at 203.2 97.79 0)
 			(hide yes)
@@
 		)
 		(instances
-			(project "skilleye"
+			(project "skilleye_1.0"
 				(path "/e922ced9-cce7-4ffa-8992-2bb79546169b/772fd356-96ac-42b2-8558-9fa39f1e8a4f"
 					(reference "R4")
@@
 			)
 		)
-		(property "Footprint" ""
+		(property "Footprint" "Resistor_SMD:R_0805_2012Metric"
 			(at 132.08 92.71 0)
 			(hide yes)
@@
 		)
 		(instances
-			(project "skilleye"
+			(project "skilleye_1.0"
 				(path "/e922ced9-cce7-4ffa-8992-2bb79546169b/772fd356-96ac-42b2-8558-9fa39f1e8a4f"
 					(reference "R3")
@@
 			)
 		)
-		(property "Footprint" ""
+		(property "Footprint" "Resistor_SMD:R_0805_2012Metric"
 			(at 233.68 97.79 0)
 			(hide yes)
@@
 		)
 		(instances
-			(project "skilleye"
+			(project "skilleye_1.0"
 				(path "/e922ced9-cce7-4ffa-8992-2bb79546169b/772fd356-96ac-42b2-8558-9fa39f1e8a4f"
 					(reference "R2")
@@
 			)
 		)
-		(property "Footprint" ""
+		(property "Footprint" "Capacitor_SMD:C_0805_2012Metric"
 			(at 262.89 97.79 0)
 			(hide yes)
@@
 		)
 		(instances
-			(project "skilleye"
+			(project "skilleye_1.0"
 				(path "/e922ced9-cce7-4ffa-8992-2bb79546169b/772fd356-96ac-42b2-8558-9fa39f1e8a4f"
 					(reference "C1")
@@
 			)
 		)
-		(property "Footprint" "Package_SO:SOIC-8-1EP_3.9x4.9mm_P1.27mm_EP2.41x3.3mm_ThermalVias"
+		(property "Footprint" "Package_SO:SOIC-8-1EP_3.9x4.9mm_P1.27mm_EP2.41x3.81mm"
 			(at 218.948 120.65 0)
 			(hide yes)
@@
 		)
 		(instances
-			(project "skilleye"
+			(project "skilleye_1.0"
 				(path "/e922ced9-cce7-4ffa-8992-2bb79546169b/772fd356-96ac-42b2-8558-9fa39f1e8a4f"
 					(reference "U1")
@@
 			)
 		)
-		(property "Footprint" ""
+		(property "Footprint" "LED_SMD:LED_0805_2012Metric"
 			(at 195.58 97.79 90)
 			(hide yes)
@@
 		)
 		(instances
-			(project "skilleye"
+			(project "skilleye_1.0"
 				(path "/e922ced9-cce7-4ffa-8992-2bb79546169b/772fd356-96ac-42b2-8558-9fa39f1e8a4f"
 					(reference "D1")
@@
 			)
 		)
-		(property "Footprint" ""
+		(property "Footprint" "Resistor_SMD:R_0805_2012Metric"
 			(at 203.2 100.33 0)
 			(hide yes)
@@
 		)
 		(instances
-			(project "skilleye"
+			(project "skilleye_1.0"
 				(path "/e922ced9-cce7-4ffa-8992-2bb79546169b/772fd356-96ac-42b2-8558-9fa39f1e8a4f"
 					(reference "R5")
@@
 			)
 		)
-		(property "Footprint" ""
+		(property "Footprint" "Connector_PinHeader_2.54mm:PinHeader_1x02_P2.54mm_Vertical"
 			(at 41.91 97.79 0)
 			(hide yes)
@@
 		)
 		(instances
-			(project "skilleye"
+			(project "skilleye_1.0"
 				(path "/e922ced9-cce7-4ffa-8992-2bb79546169b/772fd356-96ac-42b2-8558-9fa39f1e8a4f"
 					(reference "J1")
@@
 			)
 		)
-		(property "Footprint" ""
+		(property "Footprint" "Resistor_SMD:R_0805_2012Metric"
 			(at 165.1 101.6 0)
 			(hide yes)
@@
 		)
 		(instances
-			(project "skilleye"
+			(project "skilleye_1.0"
 				(path "/e922ced9-cce7-4ffa-8992-2bb79546169b/772fd356-96ac-42b2-8558-9fa39f1e8a4f"
 					(reference "R6")
@@
 		)
 		(instances
-			(project "skilleye"
+			(project "skilleye_1.0"
 				(path "/e922ced9-cce7-4ffa-8992-2bb79546169b/772fd356-96ac-42b2-8558-9fa39f1e8a4f"
 					(reference "#PWR03")
@@
 		)
 		(instances
-			(project "skilleye"
+			(project "skilleye_1.0"
 				(path "/e922ced9-cce7-4ffa-8992-2bb79546169b/772fd356-96ac-42b2-8558-9fa39f1e8a4f"
 					(reference "#PWR06")
@@
 			)
 		)
-		(property "Footprint" ""
+		(property "Footprint" "LED_SMD:LED_0805_2012Metric"
 			(at 195.58 100.33 90)
 			(hide yes)
@@
 		)
 		(instances
-			(project "skilleye"
+			(project "skilleye_1.0"
 				(path "/e922ced9-cce7-4ffa-8992-2bb79546169b/772fd356-96ac-42b2-8558-9fa39f1e8a4f"
 					(reference "D2")
@@
 			)
 		)
-		(property "Footprint" ""
+		(property "Footprint" "FS8205A:SOP65P640X120-8N"
 			(at 91.44 101.6 0)
 			(hide yes)
@@
 		)
 		(instances
-			(project "skilleye"
+			(project "skilleye_1.0"
 				(path "/e922ced9-cce7-4ffa-8992-2bb79546169b/772fd356-96ac-42b2-8558-9fa39f1e8a4f"
 					(reference "Q1")
@@
 		)
 		(instances
-			(project "skilleye"
+			(project "skilleye_1.0"
 				(path "/e922ced9-cce7-4ffa-8992-2bb79546169b/772fd356-96ac-42b2-8558-9fa39f1e8a4f"
 					(reference "#PWR02")
@@
 			)
 		)
-		(property "Footprint" ""
+		(property "Footprint" "Capacitor_SMD:C_0805_2012Metric"
 			(at 134.62 99.06 0)
 			(hide yes)
@@
 		)
 		(instances
-			(project "skilleye"
+			(project "skilleye_1.0"
 				(path "/e922ced9-cce7-4ffa-8992-2bb79546169b/772fd356-96ac-42b2-8558-9fa39f1e8a4f"
 					(reference "C3")
@@
 		)
 		(instances
-			(project "skilleye"
+			(project "skilleye_1.0"
 				(path "/e922ced9-cce7-4ffa-8992-2bb79546169b/772fd356-96ac-42b2-8558-9fa39f1e8a4f"
 					(reference "#FLG03")
@@
 		)
 		(instances
-			(project "skilleye"
+			(project "skilleye_1.0"
 				(path "/e922ced9-cce7-4ffa-8992-2bb79546169b/772fd356-96ac-42b2-8558-9fa39f1e8a4f"
 					(reference "#PWR020")
@@
 			)
 		)
-		(property "Footprint" ""
+		(property "Footprint" "Capacitor_SMD:C_0805_2012Metric"
 			(at 247.65 96.52 0)
 			(hide yes)
@@
 		)
 		(instances
-			(project "skilleye"
+			(project "skilleye_1.0"
 				(path "/e922ced9-cce7-4ffa-8992-2bb79546169b/772fd356-96ac-42b2-8558-9fa39f1e8a4f"
 					(reference "C2")
@@
 			)
 		)
-		(property "Footprint" ""
+		(property "Footprint" "Resistor_SMD:R_0805_2012Metric"
 			(at 233.68 100.33 0)
 			(hide yes)
@@
 		)
 		(instances
-			(project "skilleye"
+			(project "skilleye_1.0"
 				(path "/e922ced9-cce7-4ffa-8992-2bb79546169b/772fd356-96ac-42b2-8558-9fa39f1e8a4f"
 					(reference "R1")
@@
 		)
 		(instances
-			(project "skilleye"
+			(project "skilleye_1.0"
 				(path "/e922ced9-cce7-4ffa-8992-2bb79546169b/772fd356-96ac-42b2-8558-9fa39f1e8a4f"
 					(reference "#PWR04")
@@
 		)
 		(instances
-			(project "skilleye"
+			(project "skilleye_1.0"
 				(path "/e922ced9-cce7-4ffa-8992-2bb79546169b/772fd356-96ac-42b2-8558-9fa39f1e8a4f"
 					(reference "#FLG04")
@@
 		)
 		(instances
-			(project "skilleye"
+			(project "skilleye_1.0"
 				(path "/e922ced9-cce7-4ffa-8992-2bb79546169b/772fd356-96ac-42b2-8558-9fa39f1e8a4f"
 					(reference "#FLG05")
@@
 		)
 		(instances
-			(project "skilleye"
+			(project "skilleye_1.0"
 				(path "/e922ced9-cce7-4ffa-8992-2bb79546169b/772fd356-96ac-42b2-8558-9fa39f1e8a4f"
 					(reference "#FLG01")
@@
 		)
 		(instances
-			(project "skilleye"
+			(project "skilleye_1.0"
 				(path "/e922ced9-cce7-4ffa-8992-2bb79546169b/772fd356-96ac-42b2-8558-9fa39f1e8a4f"
 					(reference "#PWR05")
@@
 		)
 		(instances
-			(project "skilleye"
+			(project "skilleye_1.0"
 				(path "/e922ced9-cce7-4ffa-8992-2bb79546169b/772fd356-96ac-42b2-8558-9fa39f1e8a4f"
 					(reference "U2")
@@
 		)
 		(instances
-			(project "skilleye"
+			(project "skilleye_1.0"
 				(path "/e922ced9-cce7-4ffa-8992-2bb79546169b/772fd356-96ac-42b2-8558-9fa39f1e8a4f"
 					(reference "#PWR025")
