File: hardware/skilleye_1.0/skilleye_mcu.kicad_sch (KiCad schematic)
At the start: 20 parts, among them SW1 SW_Push_45deg, SW2 SW_Push_45deg, U4 ESP32-C6-WROOM-1 (N8), U5 LSM6DS0

Commit message: added 2.0 schematic
Parts:
- C10, C6, C7, C8, C9: footprint (none) -> Capacitor_SMD:C_0805_2012Metric
- R10, R13, R14, R7, R8, R9: footprint (none) -> Resistor_SMD:R_0805_2012Metric
- TP1, TP2, TP3, TP4, TP5: footprint (none) -> TestPoint:TestPoint_Pad_D1.5mm
Changed lines of the file:
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@@
 			)
 		)
-		(property "Footprint" ""
+		(property "Footprint" "Capacitor_SMD:C_0805_2012Metric"
 			(at 73.66 67.31 0)
 			(hide yes)
@@
 		)
 		(instances
-			(project "skilleye"
+			(project "skilleye_1.0"
 				(path "/e922ced9-cce7-4ffa-8992-2bb79546169b/eeb8364d-fb88-4868-b54f-166d620b4179"
 					(reference "C6")
@@
 			)
 		)
-		(property "Footprint" ""
+		(property "Footprint" "Capacitor_SMD:C_0805_2012Metric"
 			(at 196.85 102.87 0)
 			(hide yes)
@@
 		)
 		(instances
-			(project "skilleye"
+			(project "skilleye_1.0"
 				(path "/e922ced9-cce7-4ffa-8992-2bb79546169b/eeb8364d-fb88-4868-b54f-166d620b4179"
 					(reference "C10")
@@
 			)
 		)
-		(property "Footprint" ""
+		(property "Footprint" "Resistor_SMD:R_0805_2012Metric"
 			(at 158.75 138.43 0)
 			(hide yes)
@@
 		)
 		(instances
-			(project "skilleye"
+			(project "skilleye_1.0"
 				(path "/e922ced9-cce7-4ffa-8992-2bb79546169b/eeb8364d-fb88-4868-b54f-166d620b4179"
 					(reference "R14")
@@
 		)
 		(instances
-			(project "skilleye"
+			(project "skilleye_1.0"
 				(path "/e922ced9-cce7-4ffa-8992-2bb79546169b/eeb8364d-fb88-4868-b54f-166d620b4179"
 					(reference "#PWR027")
@@
 		)
 		(instances
-			(project "skilleye"
+			(project "skilleye_1.0"
 				(path "/e922ced9-cce7-4ffa-8992-2bb79546169b/eeb8364d-fb88-4868-b54f-166d620b4179"
 					(reference "U4")
@@
 		)
 		(instances
-			(project "skilleye"
+			(project "skilleye_1.0"
 				(path "/e922ced9-cce7-4ffa-8992-2bb79546169b/eeb8364d-fb88-4868-b54f-166d620b4179"
 					(reference "#PWR026")
@@
 		)
 		(instances
-			(project "skilleye"
+			(project "skilleye_1.0"
 				(path "/e922ced9-cce7-4ffa-8992-2bb79546169b/eeb8364d-fb88-4868-b54f-166d620b4179"
 					(reference "#PWR019")
@@
 		)
 		(instances
-			(project "skilleye"
+			(project "skilleye_1.0"
 				(path "/e922ced9-cce7-4ffa-8992-2bb79546169b/eeb8364d-fb88-4868-b54f-166d620b4179"
 					(reference "#PWR015")
@@
 			)
 		)
-		(property "Footprint" ""
+		(property "Footprint" "TestPoint:TestPoint_Pad_D1.5mm"
 			(at 161.29 123.19 0)
 			(hide yes)
@@
 		)
 		(instances
-			(project "skilleye"
+			(project "skilleye_1.0"
 				(path "/e922ced9-cce7-4ffa-8992-2bb79546169b/eeb8364d-fb88-4868-b54f-166d620b4179"
 					(reference "TP5")
@@
 			)
 		)
-		(property "Footprint" ""
+		(property "Footprint" "Resistor_SMD:R_0805_2012Metric"
 			(at 255.27 99.06 0)
 			(hide yes)
@@
 		)
 		(instances
-			(project "skilleye"
+			(project "skilleye_1.0"
 				(path "/e922ced9-cce7-4ffa-8992-2bb79546169b/eeb8364d-fb88-4868-b54f-166d620b4179"
 					(reference "R10")
@@
 			)
 		)
-		(property "Footprint" ""
+		(property "Footprint" "Capacitor_SMD:C_0805_2012Metric"
 			(at 73.66 62.23 0)
 			(hide yes)
@@
 		)
 		(instances
-			(project "skilleye"
+			(project "skilleye_1.0"
 				(path "/e922ced9-cce7-4ffa-8992-2bb79546169b/eeb8364d-fb88-4868-b54f-166d620b4179"
 					(reference "C7")
@@
 			)
 		)
-		(property "Footprint" ""
+		(property "Footprint" "Resistor_SMD:R_0805_2012Metric"
 			(at 158.75 97.79 0)
 			(hide yes)
@@
 		)
 		(instances
-			(project "skilleye"
+			(project "skilleye_1.0"
 				(path "/e922ced9-cce7-4ffa-8992-2bb79546169b/eeb8364d-fb88-4868-b54f-166d620b4179"
 					(reference "R8")
@@
 			)
 		)
-		(property "Footprint" ""
+		(property "Footprint" "TestPoint:TestPoint_Pad_D1.5mm"
 			(at 143.51 77.47 0)
 			(hide yes)
@@
 		)
 		(instances
-			(project "skilleye"
+			(project "skilleye_1.0"
 				(path "/e922ced9-cce7-4ffa-8992-2bb79546169b/eeb8364d-fb88-4868-b54f-166d620b4179"
 					(reference "TP1")
@@
 			)
 		)
-		(property "Footprint" ""
+		(property "Footprint" "Capacitor_SMD:C_0805_2012Metric"
 			(at 200.66 102.87 0)
 			(hide yes)
@@
 		)
 		(instances
-			(project "skilleye"
+			(project "skilleye_1.0"
 				(path "/e922ced9-cce7-4ffa-8992-2bb79546169b/eeb8364d-fb88-4868-b54f-166d620b4179"
 					(reference "C9")
@@
 			)
 		)
-		(property "Footprint" ""
+		(property "Footprint" "Resistor_SMD:R_0805_2012Metric"
 			(at 54.61 77.47 0)
 			(hide yes)
@@
 		)
 		(instances
-			(project "skilleye"
+			(project "skilleye_1.0"
 				(path "/e922ced9-cce7-4ffa-8992-2bb79546169b/eeb8364d-fb88-4868-b54f-166d620b4179"
 					(reference "R7")
@@
 		)
 		(instances
-			(project "skilleye"
+			(project "skilleye_1.0"
 				(path "/e922ced9-cce7-4ffa-8992-2bb79546169b/eeb8364d-fb88-4868-b54f-166d620b4179"
 					(reference "U5")
@@
 		)
 		(instances
-			(project "skilleye"
+			(project "skilleye_1.0"
 				(path "/e922ced9-cce7-4ffa-8992-2bb79546169b/eeb8364d-fb88-4868-b54f-166d620b4179"
 					(reference "#PWR017")
@@
 		)
 		(instances
-			(project "skilleye"
+			(project "skilleye_1.0"
 				(path "/e922ced9-cce7-4ffa-8992-2bb79546169b/eeb8364d-fb88-4868-b54f-166d620b4179"
 					(reference "SW1")
@@
 			)
 		)
-		(property "Footprint" ""
+		(property "Footprint" "Resistor_SMD:R_0805_2012Metric"
 			(at 158.75 135.89 0)
 			(hide yes)
@@
 		)
 		(instances
-			(project "skilleye"
+			(project "skilleye_1.0"
 				(path "/e922ced9-cce7-4ffa-8992-2bb79546169b/eeb8364d-fb88-4868-b54f-166d620b4179"
 					(reference "R13")
@@
 			)
 		)
-		(property "Footprint" ""
+		(property "Footprint" "TestPoint:TestPoint_Pad_D1.5mm"
 			(at 77.47 87.63 0)
 			(hide yes)
@@
 		)
 		(instances
-			(project "skilleye"
+			(project "skilleye_1.0"
 				(path "/e922ced9-cce7-4ffa-8992-2bb79546169b/eeb8364d-fb88-4868-b54f-166d620b4179"
 					(reference "TP3")
@@
 			)
 		)
-		(property "Footprint" ""
+		(property "Footprint" "Capacitor_SMD:C_0805_2012Metric"
 			(at 54.61 81.28 0)
 			(hide yes)
@@
 		)
 		(instances
-			(project "skilleye"
+			(project "skilleye_1.0"
 				(path "/e922ced9-cce7-4ffa-8992-2bb79546169b/eeb8364d-fb88-4868-b54f-166d620b4179"
 					(reference "C8")
@@
 			)
 		)
-		(property "Footprint" ""
+		(property "Footprint" "TestPoint:TestPoint_Pad_D1.5mm"
 			(at 143.51 80.01 0)
 			(hide yes)
@@
 		)
 		(instances
-			(project "skilleye"
+			(project "skilleye_1.0"
 				(path "/e922ced9-cce7-4ffa-8992-2bb79546169b/eeb8364d-fb88-4868-b54f-166d620b4179"
 					(reference "TP2")
@@
 		)
 		(instances
-			(project "skilleye"
+			(project "skilleye_1.0"
 				(path "/e922ced9-cce7-4ffa-8992-2bb79546169b/eeb8364d-fb88-4868-b54f-166d620b4179"
 					(reference "#PWR012")
@@
 		)
 		(instances
-			(project "skilleye"
+			(project "skilleye_1.0"
 				(path "/e922ced9-cce7-4ffa-8992-2bb79546169b/eeb8364d-fb88-4868-b54f-166d620b4179"
 					(reference "#PWR016")
@@
 			)
 		)
-		(property "Footprint" ""
+		(property "Footprint" "TestPoint:TestPoint_Pad_D1.5mm"
 			(at 77.47 90.17 0)
 			(hide yes)
@@
 		)
 		(instances
-			(project "skilleye"
+			(project "skilleye_1.0"
 				(path "/e922ced9-cce7-4ffa-8992-2bb79546169b/eeb8364d-fb88-4868-b54f-166d620b4179"
 					(reference "TP4")
@@
 		)
 		(instances
-			(project "skilleye"
+			(project "skilleye_1.0"
 				(path "/e922ced9-cce7-4ffa-8992-2bb79546169b/eeb8364d-fb88-4868-b54f-166d620b4179"
 					(reference "#PWR09")
@@
 		)
 		(instances
-			(project "skilleye"
+			(project "skilleye_1.0"
 				(path "/e922ced9-cce7-4ffa-8992-2bb79546169b/eeb8364d-fb88-4868-b54f-166d620b4179"
 					(reference "#PWR010")
@@
 		)
 		(instances
-			(project "skilleye"
+			(project "skilleye_1.0"
 				(path "/e922ced9-cce7-4ffa-8992-2bb79546169b/eeb8364d-fb88-4868-b54f-166d620b4179"
 					(reference "#PWR018")
@@
 		)
 		(instances
-			(project "skilleye"
+			(project "skilleye_1.0"
 				(path "/e922ced9-cce7-4ffa-8992-2bb79546169b/eeb8364d-fb88-4868-b54f-166d620b4179"
 					(reference "#PWR013")
@@
 		)
 		(instances
-			(project "skilleye"
+			(project "skilleye_1.0"
 				(path "/e922ced9-cce7-4ffa-8992-2bb79546169b/eeb8364d-fb88-4868-b54f-166d620b4179"
 					(reference "#PWR014")
@@
 			)
 		)
-		(property "Footprint" ""
+		(property "Footprint" "Resistor_SMD:R_0805_2012Metric"
 			(at 158.75 100.33 0)
 			(hide yes)
@@
 		)
 		(instances
-			(project "skilleye"
+			(project "skilleye_1.0"
 				(path "/e922ced9-cce7-4ffa-8992-2bb79546169b/eeb8364d-fb88-4868-b54f-166d620b4179"
 					(reference "R9")
@@
 		)
 		(instances
-			(project "skilleye"
+			(project "skilleye_1.0"
 				(path "/e922ced9-cce7-4ffa-8992-2bb79546169b/eeb8364d-fb88-4868-b54f-166d620b4179"
 					(reference "#PWR011")
@@
 		)
 		(instances
-			(project "skilleye"
+			(project "skilleye_1.0"
 				(path "/e922ced9-cce7-4ffa-8992-2bb79546169b/eeb8364d-fb88-4868-b54f-166d620b4179"
 					(reference "SW2")
