File: hardware/skilleye_1.0/skilleye_regulator.kicad_sch (KiCad schematic)
At the start: 3 parts, among them U3 HT7833

Commit message: added 2.0 schematic
Parts:
- C4, C5: footprint (none) -> Capacitor_SMD:C_0805_2012Metric
Changed lines of the file:
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@@
 			)
 		)
-		(property "Footprint" ""
+		(property "Footprint" "Capacitor_SMD:C_0805_2012Metric"
 			(at 152.4 105.41 0)
 			(hide yes)
@@
 		)
 		(instances
-			(project "skilleye"
+			(project "skilleye_1.0"
 				(path "/e922ced9-cce7-4ffa-8992-2bb79546169b/331d9fae-dc89-4e08-93fe-26225e9367f3"
 					(reference "C5")
@@
 		)
 		(instances
-			(project "skilleye"
+			(project "skilleye_1.0"
 				(path "/e922ced9-cce7-4ffa-8992-2bb79546169b/331d9fae-dc89-4e08-93fe-26225e9367f3"
 					(reference "#PWR08")
@@
 		)
 		(instances
-			(project "skilleye"
+			(project "skilleye_1.0"
 				(path "/e922ced9-cce7-4ffa-8992-2bb79546169b/331d9fae-dc89-4e08-93fe-26225e9367f3"
 					(reference "#PWR07")
@@
 			)
 		)
-		(property "Footprint" ""
+		(property "Footprint" "Capacitor_SMD:C_0805_2012Metric"
 			(at 139.7 105.41 0)
 			(hide yes)
@@
 		)
 		(instances
-			(project "skilleye"
+			(project "skilleye_1.0"
 				(path "/e922ced9-cce7-4ffa-8992-2bb79546169b/331d9fae-dc89-4e08-93fe-26225e9367f3"
 					(reference "C4")
@@
 		)
 		(instances
-			(project "skilleye"
+			(project "skilleye_1.0"
 				(path "/e922ced9-cce7-4ffa-8992-2bb79546169b/331d9fae-dc89-4e08-93fe-26225e9367f3"
 					(reference "U3")
