File: hardware/skilleye_2.0/skilleye_2.0.kicad_sch (KiCad schematic)
At the start: 4 parts, among them J1 TP4056 Breakout, U1 XIAO-ESP32-C6-SMD, U2 GY-521

Commit message: added 2.0 pcb layout
Parts:
- added SW1: SW_SPDT, Button_Switch_THT:SW_Slide_SPDT_Straight_CK_OS102011MS2Q, symbol Switch:SW_SPDT
Connections:
- net BATT+: now reaches BT1.1 (+), J1.3 (B+)
- net BATT-: now reaches BT1.2 (-), J1.4 (B-)
- net VBAT_RAW: now reaches J1.5 (OUT+)
- net VBAT_RAW: now also SW1.2 (B); no longer U1.23 (VBAT)
- net IMU_INT: now reaches U2.INT
- net IMU_INT: now also U1.1 (D0)
- new net VBAT_SW: SW1.1 (A), U1.23 (VBAT)
- no-connect marks 21 -> 20
Changed lines of the file:
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@@
 	(title_block
 		(title "Skilleye")
-		(date "2026-07-25")
-		(rev "2.0")
+		(date "2026-07-27")
+		(rev "2.1")
 		(company "National Taipei University of Technology - Dept. of EECS")
 		(comment 1 "SkillEye")
@@
 	)
 	(no_connect
+		(at 99.06 124.46)
+	)
+	(no_connect
 		(at 133.35 80.01)
 	)
@@
 	)
 	(no_connect
-		(at 222.25 99.06)
-	)
-	(no_connect
 		(at 148.59 80.01)
 	)
@@
 	)
 	(no_connect
-		(at 118.11 91.44)
-	)
-	(no_connect
 		(at 129.54 80.01)
 	)
@@
 	(wire
 		(pts
-			(xy 95.25 124.46) (xy 137.16 124.46)
-		)
-		(stroke
-			(width 0)
-			(type default)
-		)
-	)
-	(wire
-		(pts
 			(xy 91.44 101.6) (xy 91.44 102.87)
 		)
@@
 	(wire
 		(pts
+			(xy 101.6 96.52) (xy 101.6 114.3)
+		)
+		(stroke
+			(width 0)
+			(type default)
+		)
+	)
+	(wire
+		(pts
 			(xy 81.28 114.3) (xy 82.55 114.3)
 		)
@@
 	(wire
 		(pts
-			(xy 95.25 96.52) (xy 95.25 124.46)
-		)
-		(stroke
-			(width 0)
-			(type default)
-		)
-	)
-	(wire
-		(pts
 			(xy 72.39 114.3) (xy 72.39 109.22)
 		)
@@
 	(wire
 		(pts
+			(xy 104.14 124.46) (xy 137.16 124.46)
+		)
+		(stroke
+			(width 0)
+			(type default)
+		)
+	)
+	(wire
+		(pts
 			(xy 223.52 111.76) (xy 223.52 113.03)
 		)
@@
 	(wire
 		(pts
-			(xy 90.17 96.52) (xy 95.25 96.52)
-		)
-		(stroke
-			(width 0)
-			(type default)
-		)
-	)
-	(wire
-		(pts
 			(xy 184.15 99.06) (xy 191.77 99.06)
 		)
@@
 	(wire
 		(pts
+			(xy 90.17 96.52) (xy 101.6 96.52)
+		)
+		(stroke
+			(width 0)
+			(type default)
+		)
+	)
+	(wire
+		(pts
 			(xy 223.52 93.98) (xy 223.52 92.71)
 		)
@@
 			(width 0)
 			(type default)
+		)
+	)
+	(label "IMU_INT"
+		(at 222.25 99.06 0)
+		(effects
+			(font
+				(size 1.27 1.27)
+			)
+			(justify left bottom)
+		)
+	)
+	(label "VBAT_RAW"
+		(at 92.71 96.52 0)
+		(effects
+			(font
+				(size 1.27 1.27)
+			)
+			(justify left bottom)
 		)
 	)
@@
 		)
 	)
+	(label "IMU_INT"
+		(at 118.11 91.44 180)
+		(effects
+			(font
+				(size 1.27 1.27)
+			)
+			(justify right bottom)
+		)
+	)
+	(label "VBAT_SW"
+		(at 121.92 124.46 180)
+		(effects
+			(font
+				(size 1.27 1.27)
+			)
+			(justify right bottom)
+		)
+	)
 	(label "SCL"
 		(at 191.77 104.14 180)
@@
 		)
 	)
+	(label "BATT-"
+		(at 82.55 114.3 0)
+		(effects
+			(font
+				(size 1.27 1.27)
+			)
+			(justify left bottom)
+		)
+	)
 	(label "SDA"
 		(at 118.11 106.68 180)
@@
 	(label "SCL"
 		(at 118.11 110.49 180)
+		(effects
+			(font
+				(size 1.27 1.27)
+			)
+			(justify right bottom)
+		)
+	)
+	(label "BATT+"
+		(at 72.39 114.3 180)
 		(effects
 			(font
@@
 					(unit 1)
 				)
+			)
+		)
+	)
+	(symbol
+		(lib_id "Switch:SW_SPDT")
+		(at 101.6 119.38 270)
+		(unit 1)
+		(body_style 1)
+		(exclude_from_sim no)
+		(in_bom yes)
+		(on_board yes)
+		(in_pos_files yes)
+		(dnp no)
+		(fields_autoplaced yes)
+		(property "Reference" "SW1"
+			(at 106.68 118.1099 90)
+			(show_name no)
+			(do_not_autoplace no)
+			(effects
+				(font
+					(size 1.27 1.27)
+				)
+				(justify left)
+			)
+		)
+		(property "Value" "SW_SPDT"
+			(at 106.68 120.6499 90)
+			(show_name no)
+			(do_not_autoplace no)
+			(effects
+				(font
+					(size 1.27 1.27)
+				)
+				(justify left)
+			)
+		)
+		(property "Footprint" "Button_Switch_THT:SW_Slide_SPDT_Straight_CK_OS102011MS2Q"
+			(at 101.6 119.38 0)
+			(hide yes)
+			(show_name no)
+			(do_not_autoplace no)
+			(effects
+				(font
+					(size 1.27 1.27)
+				)
+			)
+		)
+		(property "Datasheet" ""
+			(at 93.98 119.38 0)
+			(hide yes)
+			(show_name no)
+			(do_not_autoplace no)
+			(effects
+				(font
+					(size 1.27 1.27)
+				)
+			)
+		)
+		(property "Description" "Switch, single pole double throw"
+			(at 101.6 119.38 0)
+			(hide yes)
+			(show_name no)
+			(do_not_autoplace no)
+			(effects
+				(font
+					(size 1.27 1.27)
+				)
+			)
+		)
+		(pin "2"
+		)
+		(pin "1"
+		)
+		(pin "3"
+		)
+		(instances
+			(project "skilleye_2.0"
+				(path "/d8a7564c-1896-4459-8d91-f745b165ebeb"
+					(reference "SW1")
+					(unit 1)
+				)

Commit message: layout update for fabrication constraints
Other:
- title: Skilleye -> SkillEye
Changed lines of the file:
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@@
 	(paper "A4")
 	(title_block
-		(title "Skilleye")
+		(title "SkillEye")
 		(date "2026-07-27")
 		(rev "2.1")
 		(company "National Taipei University of Technology - Dept. of EECS")
-		(comment 1 "SkillEye")
-		(comment 2 "Designer: Purit Hongjirakul")
-		(comment 3 "https://github.com/rizalfanex/SkillEye")
+		(comment 1 "Designer: Purit Hongjirakul")
+		(comment 2 "https://github.com/rizalfanex/SkillEye")
 	)
 	(junction
